File: bifrost.kicad_pcb (KiCad board)
At the start: 2 copper layers, 73.7 x 71.1 mm, 77 parts, among them J1 395430002, J10 Conn_0.1_01x04, J11 Conn_0.1_01x06, J12 Micro_SD_Card_Det_Single, J2 395430002, J3 393570003, J4 393570003, J5 393570003, J6 393570003, J7 SJ_3524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

Commit message: Move logos around
Parts:
- moved G*** 1.27 mm to (161.9, 73.0)
- moved G*** 0.63 mm to (156.8, 74.9)
Changed lines of the file:
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@@
   )
   (module bifrost-logo:bifrost (layer F.Cu)
-    (at 160.655 73.025)
+    (at 161.925 73.025)
     (fp_text reference G*** (at 0 0) (layer F.SilkS) hide
       (effects (font (size 1.524 1.524) (thickness 0.3)))
@@
   )
   (module bifrost-logo:rrwb (layer B.Cu)
-    (at 157.48 74.93 180)
+    (at 156.845 74.93 180)
     (fp_text reference G*** (at 0 0) (layer B.SilkS) hide
       (effects (font (size 1.524 1.524) (thickness 0.3)) (justify mirror))

Commit message: Clean up
Parts:
- turned C10 to 90 degrees
- turned C9 to 90 degrees
Routing:
- net +3V3: track 31.0 -> 35.3 mm
- net Net-(J12-Pad3): track 26.2 -> 30.2 mm
- net GND: track 22.4 -> 23.9 mm
- net /BTN1: track 42.5 -> 41.8 mm
- net /BTN2: track 41.4 -> 40.7 mm
- net /BTN3: track 55.9 -> 56.5 mm
Other:
- board text added: "JLCJLCJLCJLC"
