File: bifrost.kicad_pcb (KiCad board)
At the start: 2 copper layers, 73.7 x 71.1 mm, 78 parts, among them J1 395430002, J10 Conn_0.1_01x04, J11 Conn_0.1_01x06, J12 Micro_SD_Card_Det_Single, J13 Conn_03x07_23_Common, J2 395430002, J3 393570003, J4 393570003, J5 393570003, J6 393570003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

Commit message: Complete routing
Parts:
- moved D3 0.64 mm to (156.8, 111.1)
- moved D4 0.64 mm to (160.7, 111.1)
- moved D5 0.64 mm to (164.5, 111.1)
- moved R16 0.64 mm to (156.8, 111.1)
- moved R17 0.64 mm to (160.7, 111.1)
- moved R18 0.64 mm to (164.5, 111.1)
Routing:
- net +5V: track 207.1 -> 238.0 mm, vias 8 -> 9
- net /BTN1: track 41.8 -> 71.4 mm, vias 0 -> 1
- net /BTN3: track 56.5 -> 72.6 mm
- net /LED3: track 11.6 -> 24.4 mm
- net /BTN2: track 40.7 -> 53.3 mm
- net /BTN4: track 69.5 -> 81.7 mm
- net /LED1: track 13.9 -> 24.4 mm
- net /LED2: track 10.5 -> 20.9 mm
- net /AUD_L: track 27.5 -> 32.4 mm
